File: flowstick_led_strip_pcbs/strip.kicad_sch (KiCad schematic)
At the start: 45 parts

Commit message: work on rev2 + panelize LED strips
Parts:
- added H1, H3, H5: MountingHole_Pad, custom:single_b2b_pad_doublewide, symbol Mechanical:MountingHole_Pad
Connections:
- net +5V: now also H1.1, H3.1, H5.1

Commit message: Update LED strips to use to 6-pin LED package
Parts:
- D1, D10, D11, D12, D13, D14, D15, D16, D17, D18, D19, D2, D20, D21, D22, D23, D24, D25, D26, D27, D28, D29, D3, D30, D31, D32, D33, D34, D35, D36, D37, D38, D39, D4, D40, D5, D6, D7, D8, D9: footprint LED_SMD:LED-APA102-2020 -> custom:LED-APA102-2020-6
Changed lines of the file:
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@@
 			)
 		)
-		(property "Footprint" "LED_SMD:LED-APA102-2020"
+		(property "Footprint" "custom:LED-APA102-2020-6"
 			(at 161.29 60.96 0)
 			(effects
@@
 			)
 		)
-		(property "Footprint" "LED_SMD:LED-APA102-2020"
+		(property "Footprint" "custom:LED-APA102-2020-6"
 			(at 161.29 124.46 0)
 			(effects
@@
 			)
 		)
-		(property "Footprint" "LED_SMD:LED-APA102-2020"
+		(property "Footprint" "custom:LED-APA102-2020-6"
 			(at 115.57 156.21 0)
 			(effects
@@
 			)
 		)
-		(property "Footprint" "LED_SMD:LED-APA102-2020"
+		(property "Footprint" "custom:LED-APA102-2020-6"
 			(at 191.77 156.21 0)
 			(effects
@@
 			)
 		)
-		(property "Footprint" "LED_SMD:LED-APA102-2020"
+		(property "Footprint" "custom:LED-APA102-2020-6"
 			(at 69.85 124.46 0)
 			(effects
@@
 			)
 		)
-		(property "Footprint" "LED_SMD:LED-APA102-2020"
+		(property "Footprint" "custom:LED-APA102-2020-6"
 			(at 130.81 156.21 0)
 			(effects
@@
 			)
 		)
-		(property "Footprint" "LED_SMD:LED-APA102-2020"
+		(property "Footprint" "custom:LED-APA102-2020-6"
 			(at 85.09 60.96 0)
 			(effects
@@
 			)
 		)
-		(property "Footprint" "LED_SMD:LED-APA102-2020"
+		(property "Footprint" "custom:LED-APA102-2020-6"
 			(at 176.53 124.46 0)
 			(effects
@@
 			)
 		)
-		(property "Footprint" "LED_SMD:LED-APA102-2020"
+		(property "Footprint" "custom:LED-APA102-2020-6"
 			(at 69.85 92.71 0)
 			(effects
@@
 			)
 		)
-		(property "Footprint" "LED_SMD:LED-APA102-2020"
+		(property "Footprint" "custom:LED-APA102-2020-6"
 			(at 130.81 92.71 0)
 			(effects
@@
 			)
 		)
-		(property "Footprint" "LED_SMD:LED-APA102-2020"
+		(property "Footprint" "custom:LED-APA102-2020-6"
 			(at 176.53 92.71 0)
 			(effects
@@
 			)
 		)
-		(property "Footprint" "LED_SMD:LED-APA102-2020"
+		(property "Footprint" "custom:LED-APA102-2020-6"
 			(at 115.57 92.71 0)
 			(effects
@@
 			)
 		)
-		(property "Footprint" "LED_SMD:LED-APA102-2020"
+		(property "Footprint" "custom:LED-APA102-2020-6"
 			(at 191.77 60.96 0)
 			(effects
@@
 			)
 		)
-		(property "Footprint" "LED_SMD:LED-APA102-2020"
+		(property "Footprint" "custom:LED-APA102-2020-6"
 			(at 161.29 156.21 0)
 			(effects
@@
 			)
 		)
-		(property "Footprint" "LED_SMD:LED-APA102-2020"
+		(property "Footprint" "custom:LED-APA102-2020-6"
 			(at 191.77 92.71 0)
 			(effects
@@
 			)
 		)
-		(property "Footprint" "LED_SMD:LED-APA102-2020"
+		(property "Footprint" "custom:LED-APA102-2020-6"
 			(at 146.05 92.71 0)
 			(effects
@@
 			)
 		)
-		(property "Footprint" "LED_SMD:LED-APA102-2020"
+		(property "Footprint" "custom:LED-APA102-2020-6"
 			(at 100.33 92.71 0)
 			(effects
@@
 			)
 		)
-		(property "Footprint" "LED_SMD:LED-APA102-2020"
+		(property "Footprint" "custom:LED-APA102-2020-6"
 			(at 176.53 156.21 0)
 			(effects
@@
 			)
 		)
-		(property "Footprint" "LED_SMD:LED-APA102-2020"
+		(property "Footprint" "custom:LED-APA102-2020-6"
 			(at 100.33 124.46 0)
 			(effects
@@
 			)
 		)
-		(property "Footprint" "LED_SMD:LED-APA102-2020"
+		(property "Footprint" "custom:LED-APA102-2020-6"
 			(at 85.09 124.46 0)
 			(effects
@@
 			)
 		)
-		(property "Footprint" "LED_SMD:LED-APA102-2020"
+		(property "Footprint" "custom:LED-APA102-2020-6"
 			(at 54.61 60.96 0)
 			(effects
@@
 			)
 		)
-		(property "Footprint" "LED_SMD:LED-APA102-2020"
+		(property "Footprint" "custom:LED-APA102-2020-6"
 			(at 54.61 124.46 0)
 			(effects
@@
 			)
 		)
-		(property "Footprint" "LED_SMD:LED-APA102-2020"
+		(property "Footprint" "custom:LED-APA102-2020-6"
 			(at 191.77 124.46 0)
 			(effects
@@
 			)
 		)
-		(property "Footprint" "LED_SMD:LED-APA102-2020"
+		(property "Footprint" "custom:LED-APA102-2020-6"
 			(at 146.05 60.96 0)
 			(effects
@@
 			)
 		)
-		(property "Footprint" "LED_SMD:LED-APA102-2020"
+		(property "Footprint" "custom:LED-APA102-2020-6"
 			(at 54.61 156.21 0)
 			(effects
@@
 			)
 		)
-		(property "Footprint" "LED_SMD:LED-APA102-2020"
+		(property "Footprint" "custom:LED-APA102-2020-6"
 			(at 69.85 60.96 0)
 			(effects
@@
 			)
 		)
-		(property "Footprint" "LED_SMD:LED-APA102-2020"
+		(property "Footprint" "custom:LED-APA102-2020-6"
 			(at 85.09 92.71 0)
 			(effects
@@
 			)
 		)
-		(property "Footprint" "LED_SMD:LED-APA102-2020"
+		(property "Footprint" "custom:LED-APA102-2020-6"
 			(at 69.85 156.21 0)
 			(effects
@@
 			)
 		)
-		(property "Footprint" "LED_SMD:LED-APA102-2020"
+		(property "Footprint" "custom:LED-APA102-2020-6"
 			(at 130.81 124.46 0)
 			(effects
@@
 			)
 		)
-		(property "Footprint" "LED_SMD:LED-APA102-2020"
+		(property "Footprint" "custom:LED-APA102-2020-6"
 			(at 54.61 92.71 0)
 			(effects
@@
 			)
 		)
-		(property "Footprint" "LED_SMD:LED-APA102-2020"
+		(property "Footprint" "custom:LED-APA102-2020-6"
 			(at 176.53 60.96 0)
 			(effects
@@
 			)
 		)
-		(property "Footprint" "LED_SMD:LED-APA102-2020"
+		(property "Footprint" "custom:LED-APA102-2020-6"
 			(at 146.05 156.21 0)
 			(effects
@@
 			)
 		)
-		(property "Footprint" "LED_SMD:LED-APA102-2020"
+		(property "Footprint" "custom:LED-APA102-2020-6"
 			(at 115.57 60.96 0)
 			(effects
@@
 			)
 		)
-		(property "Footprint" "LED_SMD:LED-APA102-2020"
+		(property "Footprint" "custom:LED-APA102-2020-6"
 			(at 146.05 124.46 0)
 			(effects
@@
 			)
 		)
-		(property "Footprint" "LED_SMD:LED-APA102-2020"
+		(property "Footprint" "custom:LED-APA102-2020-6"
 			(at 161.29 92.71 0)
 			(effects
@@
 			)
 		)
-		(property "Footprint" "LED_SMD:LED-APA102-2020"
+		(property "Footprint" "custom:LED-APA102-2020-6"
 			(at 115.57 124.46 0)
 			(effects
@@
 			)
 		)
-		(property "Footprint" "LED_SMD:LED-APA102-2020"
+		(property "Footprint" "custom:LED-APA102-2020-6"
 			(at 130.81 60.96 0)
 			(effects
@@
 			)
 		)
-		(property "Footprint" "LED_SMD:LED-APA102-2020"
+		(property "Footprint" "custom:LED-APA102-2020-6"
 			(at 100.33 60.96 0)
 			(effects
@@
 			)
 		)
-		(property "Footprint" "LED_SMD:LED-APA102-2020"
+		(property "Footprint" "custom:LED-APA102-2020-6"
 			(at 85.09 156.21 0)
 			(effects
@@
 			)
 		)
-		(property "Footprint" "LED_SMD:LED-APA102-2020"
+		(property "Footprint" "custom:LED-APA102-2020-6"
 			(at 100.33 156.21 0)
 			(effects

Commit message: Switch to 90 degree alternate LED pinout
Parts:
- D1, D10, D11, D12, D13, D14, D15, D16, D17, D18, D19, D2, D20, D21, D22, D23, D24, D25, D26, D27, D28, D29, D3, D30, D31, D32, D33, D34, D35, D36, D37, D38, D39, D4, D40, D5, D6, D7, D8, D9: footprint custom:LED-APA102-2020-6 -> custom:LED-APA102-2020-6_90deg
Changed lines of the file:
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@@
 			)
 		)
-		(property "Footprint" "custom:LED-APA102-2020-6"
+		(property "Footprint" "custom:LED-APA102-2020-6_90deg"
 			(at 161.29 60.96 0)
 			(effects
@@
 			)
 		)
-		(property "Footprint" "custom:LED-APA102-2020-6"
+		(property "Footprint" "custom:LED-APA102-2020-6_90deg"
 			(at 161.29 124.46 0)
 			(effects
@@
 			)
 		)
-		(property "Footprint" "custom:LED-APA102-2020-6"
+		(property "Footprint" "custom:LED-APA102-2020-6_90deg"
 			(at 115.57 156.21 0)
 			(effects
@@
 			)
 		)
-		(property "Footprint" "custom:LED-APA102-2020-6"
+		(property "Footprint" "custom:LED-APA102-2020-6_90deg"
 			(at 191.77 156.21 0)
 			(effects
@@
 			)
 		)
-		(property "Footprint" "custom:LED-APA102-2020-6"
+		(property "Footprint" "custom:LED-APA102-2020-6_90deg"
 			(at 69.85 124.46 0)
 			(effects
@@
 			)
 		)
-		(property "Footprint" "custom:LED-APA102-2020-6"
+		(property "Footprint" "custom:LED-APA102-2020-6_90deg"
 			(at 130.81 156.21 0)
 			(effects
@@
 			)
 		)
-		(property "Footprint" "custom:LED-APA102-2020-6"
+		(property "Footprint" "custom:LED-APA102-2020-6_90deg"
 			(at 85.09 60.96 0)
 			(effects
@@
 			)
 		)
-		(property "Footprint" "custom:LED-APA102-2020-6"
+		(property "Footprint" "custom:LED-APA102-2020-6_90deg"
 			(at 176.53 124.46 0)
 			(effects
@@
 			)
 		)
-		(property "Footprint" "custom:LED-APA102-2020-6"
+		(property "Footprint" "custom:LED-APA102-2020-6_90deg"
 			(at 69.85 92.71 0)
 			(effects
@@
 			)
 		)
-		(property "Footprint" "custom:LED-APA102-2020-6"
+		(property "Footprint" "custom:LED-APA102-2020-6_90deg"
 			(at 130.81 92.71 0)
 			(effects
@@
 			)
 		)
-		(property "Footprint" "custom:LED-APA102-2020-6"
+		(property "Footprint" "custom:LED-APA102-2020-6_90deg"
 			(at 176.53 92.71 0)
 			(effects
@@
 			)
 		)
-		(property "Footprint" "custom:LED-APA102-2020-6"
+		(property "Footprint" "custom:LED-APA102-2020-6_90deg"
 			(at 115.57 92.71 0)
 			(effects
@@
 			)
 		)
-		(property "Footprint" "custom:LED-APA102-2020-6"
+		(property "Footprint" "custom:LED-APA102-2020-6_90deg"
 			(at 191.77 60.96 0)
 			(effects
@@
 			)
 		)
-		(property "Footprint" "custom:LED-APA102-2020-6"
+		(property "Footprint" "custom:LED-APA102-2020-6_90deg"
 			(at 161.29 156.21 0)
 			(effects
@@
 			)
 		)
-		(property "Footprint" "custom:LED-APA102-2020-6"
+		(property "Footprint" "custom:LED-APA102-2020-6_90deg"
 			(at 191.77 92.71 0)
 			(effects
@@
 			)
 		)
-		(property "Footprint" "custom:LED-APA102-2020-6"
+		(property "Footprint" "custom:LED-APA102-2020-6_90deg"
 			(at 146.05 92.71 0)
 			(effects
@@
 			)
 		)
-		(property "Footprint" "custom:LED-APA102-2020-6"
+		(property "Footprint" "custom:LED-APA102-2020-6_90deg"
 			(at 100.33 92.71 0)
 			(effects
@@
 			)
 		)
-		(property "Footprint" "custom:LED-APA102-2020-6"
+		(property "Footprint" "custom:LED-APA102-2020-6_90deg"
 			(at 176.53 156.21 0)
 			(effects
@@
 			)
 		)
-		(property "Footprint" "custom:LED-APA102-2020-6"
+		(property "Footprint" "custom:LED-APA102-2020-6_90deg"
 			(at 100.33 124.46 0)
 			(effects
@@
 			)
 		)
-		(property "Footprint" "custom:LED-APA102-2020-6"
+		(property "Footprint" "custom:LED-APA102-2020-6_90deg"
 			(at 85.09 124.46 0)
 			(effects
@@
 			)
 		)
-		(property "Footprint" "custom:LED-APA102-2020-6"
+		(property "Footprint" "custom:LED-APA102-2020-6_90deg"
 			(at 54.61 60.96 0)
 			(effects
@@
 			)
 		)
-		(property "Footprint" "custom:LED-APA102-2020-6"
+		(property "Footprint" "custom:LED-APA102-2020-6_90deg"
 			(at 54.61 124.46 0)
 			(effects
@@
 			)
 		)
-		(property "Footprint" "custom:LED-APA102-2020-6"
+		(property "Footprint" "custom:LED-APA102-2020-6_90deg"
 			(at 191.77 124.46 0)
 			(effects
@@
 			)
 		)
-		(property "Footprint" "custom:LED-APA102-2020-6"
+		(property "Footprint" "custom:LED-APA102-2020-6_90deg"
 			(at 146.05 60.96 0)
 			(effects
@@
 			)
 		)
-		(property "Footprint" "custom:LED-APA102-2020-6"
+		(property "Footprint" "custom:LED-APA102-2020-6_90deg"
 			(at 54.61 156.21 0)
 			(effects
@@
 			)
 		)
-		(property "Footprint" "custom:LED-APA102-2020-6"
+		(property "Footprint" "custom:LED-APA102-2020-6_90deg"
 			(at 69.85 60.96 0)
 			(effects
@@
 			)
 		)
-		(property "Footprint" "custom:LED-APA102-2020-6"
+		(property "Footprint" "custom:LED-APA102-2020-6_90deg"
 			(at 85.09 92.71 0)
 			(effects
@@
 			)
 		)
-		(property "Footprint" "custom:LED-APA102-2020-6"
+		(property "Footprint" "custom:LED-APA102-2020-6_90deg"
 			(at 69.85 156.21 0)
 			(effects
@@
 			)
 		)
-		(property "Footprint" "custom:LED-APA102-2020-6"
+		(property "Footprint" "custom:LED-APA102-2020-6_90deg"
 			(at 130.81 124.46 0)
 			(effects
@@
 			)
 		)
-		(property "Footprint" "custom:LED-APA102-2020-6"
+		(property "Footprint" "custom:LED-APA102-2020-6_90deg"
 			(at 54.61 92.71 0)
 			(effects
@@
 			)
 		)
-		(property "Footprint" "custom:LED-APA102-2020-6"
+		(property "Footprint" "custom:LED-APA102-2020-6_90deg"
 			(at 176.53 60.96 0)
 			(effects
@@
 			)
 		)
-		(property "Footprint" "custom:LED-APA102-2020-6"
+		(property "Footprint" "custom:LED-APA102-2020-6_90deg"
 			(at 146.05 156.21 0)
 			(effects
@@
 			)
 		)
-		(property "Footprint" "custom:LED-APA102-2020-6"
+		(property "Footprint" "custom:LED-APA102-2020-6_90deg"
 			(at 115.57 60.96 0)
 			(effects
@@
 			)
 		)
-		(property "Footprint" "custom:LED-APA102-2020-6"
+		(property "Footprint" "custom:LED-APA102-2020-6_90deg"
 			(at 146.05 124.46 0)
 			(effects
@@
 			)
 		)
-		(property "Footprint" "custom:LED-APA102-2020-6"
+		(property "Footprint" "custom:LED-APA102-2020-6_90deg"
 			(at 161.29 92.71 0)
 			(effects
@@
 			)
 		)
-		(property "Footprint" "custom:LED-APA102-2020-6"
+		(property "Footprint" "custom:LED-APA102-2020-6_90deg"
 			(at 115.57 124.46 0)
 			(effects
@@
 			)
 		)
-		(property "Footprint" "custom:LED-APA102-2020-6"
+		(property "Footprint" "custom:LED-APA102-2020-6_90deg"
 			(at 130.81 60.96 0)
 			(effects
@@
 			)
 		)
-		(property "Footprint" "custom:LED-APA102-2020-6"
+		(property "Footprint" "custom:LED-APA102-2020-6_90deg"
 			(at 100.33 60.96 0)
 			(effects
@@
 			)
 		)
-		(property "Footprint" "custom:LED-APA102-2020-6"
+		(property "Footprint" "custom:LED-APA102-2020-6_90deg"
 			(at 85.09 156.21 0)
 			(effects
@@
 			)
 		)
-		(property "Footprint" "custom:LED-APA102-2020-6"
+		(property "Footprint" "custom:LED-APA102-2020-6_90deg"
 			(at 100.33 156.21 0)
 			(effects
